File: Hardware/plus/GW5A_LV25MG121N.kicad_sch (KiCad schematic)
At the start: 31 parts, among them J1 DF40C-60DS-0.4V(51), J2 DF40C-60DS-0.4V(51), J6 Conn_01x08_Pin

Commit message: PCB修改器件干涉问题，更换LED
Parts:
- removed D1: NCD0603G1, LED_SMD:LED_0603_1608Metric, symbol HPM6280Foc:NCD0603G1
- removed D2: NCD0603R1, LED_SMD:LED_0603_1608Metric, symbol HPM6280Foc:NCD0603R1
- removed D3: NCD0603B1, LED_SMD:LED_0603_1608Metric, symbol HPM6280Foc:NCD0603B1
- added D6: LED_RGBA, Library:LED_RGBA_1615, symbol Device:LED_RGBA
Connections:
- net +3V3: now also D6.4 (A); no longer R36.1, R37.1, R38.1
- net H5_IOT61A: now also R38.2
- net J5_IOT61B: now also R37.2
- net L5_IOT63A: now also R36.2
- net MCU_SWC renamed K9_MCU_SWC
- net MCU_SWD renamed L9_MCU_SWD
- new net: D6.3 (BK), R38.1
- new net: D6.2 (GK), R37.1
- new net: D6.1 (RK), R36.1
Other:
- moved on the sheet: R36, R37, R38
