File: Hardware/plus/HFLink_Plus.kicad_pcb (KiCad board)
At the start: 4 copper layers, 48.5 x 33.5 mm, 121 parts, among them J1 DF40C-60DS-0.4V(51), J2 DF40C-60DS-0.4V(51), J3 Conn_ARM_JTAG_SWD_20, J4 USB_C_Receptacle_USB2.0_16P, J5 WAFER-ZH1.5-4PWB, J6 Conn_01x08_Pin, Q1 SI2305, U1 ECMF02-2AMX6, U10 SN74LVC1G125DCK, U11 SN74LVC1G125DCK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

Commit message: 修正串口线序
Connections:
- J5 pad 1: GND -> VTREF
- J5 pad 2: /INTERFACE/UART_RX -> /INTERFACE/UART_TX
- J5 pad 3: /INTERFACE/UART_TX -> /INTERFACE/UART_RX
- J5 pad 4: VTREF -> GND
Routing:
- net VTREF: track 67.8 -> 64.1 mm
- net /INTERFACE/UART_RX: track 23.9 -> 22.8 mm
- net /INTERFACE/UART_TX: track 29.5 -> 29.0 mm
Changed lines of the file:
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@@
 			(layers "B.Cu" "B.Mask" "B.Paste")
 			(roundrect_rratio 0.25)
-			(net 2 "GND")
+			(net 119 "VTREF")
 			(pinfunction "Pin_1")
 			(pintype "passive")
@@
 			(layers "B.Cu" "B.Mask" "B.Paste")
 			(roundrect_rratio 0.25)
-			(net 143 "/INTERFACE/UART_RX")
+			(net 144 "/INTERFACE/UART_TX")
 			(pinfunction "Pin_2")
 			(pintype "passive")
@@
 			(layers "B.Cu" "B.Mask" "B.Paste")
 			(roundrect_rratio 0.25)
-			(net 144 "/INTERFACE/UART_TX")
+			(net 143 "/INTERFACE/UART_RX")
 			(pinfunction "Pin_3")
 			(pintype "passive")
@@
 			(layers "B.Cu" "B.Mask" "B.Paste")
 			(roundrect_rratio 0.25)
-			(net 119 "VTREF")
+			(net 2 "GND")
 			(pinfunction "Pin_4")
 			(pintype "passive")
@@
 	)
 	(segment
-		(start 105.1 66.693258)
-		(end 105.1 76.05)
+		(start 96.8056 61.6169)
+		(end 99.410158 61.6169)
 		(width 0.127)
 		(layer "B.Cu")
@@
 	)
 	(segment
-		(start 104.7 76.45)
-		(end 103.225 76.45)
+		(start 104.7 71.95)
+		(end 103.225 71.95)
 		(width 0.127)
 		(layer "B.Cu")
@@
 	)
 	(segment
-		(start 102.439843 64.0331)
-		(end 105.1 66.693258)
+		(start 95.6025 62.82)
+		(end 96.8056 61.6169)
 		(width 0.127)
 		(layer "B.Cu")
@@
 	)
 	(segment
-		(start 96.8156 64.0331)
-		(end 102.439843 64.0331)
+		(start 105.2331 71.4169)
+		(end 104.7 71.95)
 		(width 0.127)
 		(layer "B.Cu")
@@
 	)
 	(segment
-		(start 105.1 76.05)
-		(end 104.7 76.45)
+		(start 105.2331 67.439842)
+		(end 105.2331 71.4169)
 		(width 0.127)
 		(layer "B.Cu")
@@
 	)
 	(segment
-		(start 95.6025 62.82)
-		(end 96.8156 64.0331)
+		(start 99.410158 61.6169)
+		(end 105.2331 67.439842)
 		(width 0.127)
 		(layer "B.Cu")
@@
 	)
 	(segment
-		(start 103.225 73.45)
-		(end 101.35 73.45)
+		(start 99.95 75.75)
+		(end 100.75 74.95)
 		(width 0.127)
 		(layer "B.Cu")
@@
 	)
 	(segment
-		(start 99.95 74.85)
+		(start 99.95 75.75)
 		(end 99.95 81.2)
 		(width 0.127)
@@
 	)
 	(segment
-		(start 101.35 73.45)
-		(end 99.95 74.85)
+		(start 100.75 74.95)
+		(end 103.225 74.95)
 		(width 0.127)
 		(layer "B.Cu")
@@
 	)
 	(segment
-		(start 94.75 64.25)
-		(end 102.35 64.25)
-		(width 0.127)
-		(layer "B.Cu")
-		(net 144)
-	)
-	(segment
-		(start 104.65 74.95)
-		(end 104.8831 74.7169)
+		(start 88.65 61)
+		(end 89.6 61.95)
 		(width 0.127)
 		(layer "B.Cu")
@@
 	)
 	(segment
-		(start 103.225 74.95)
-		(end 104.65 74.95)
+		(start 92.45 61.95)
+		(end 93 61.4)
 		(width 0.127)
 		(layer "B.Cu")
@@
 	)
 	(segment
-		(start 102.35 64.25)
-		(end 104.8831 66.7831)
+		(start 99.5 61.4)
+		(end 105.45 67.35)
 		(width 0.127)
 		(layer "B.Cu")
@@
 	)
 	(segment
-		(start 104.8831 66.7831)
-		(end 104.8831 68.05)
+		(start 93 61.4)
+		(end 99.5 61.4)
 		(width 0.127)
 		(layer "B.Cu")
@@
 	)
 	(segment
-		(start 104.8831 74.7169)
-		(end 104.8831 68)
+		(start 104.75 73.45)
+		(end 103.225 73.45)
 		(width 0.127)
 		(layer "B.Cu")
@@
 	)
 	(segment
-		(start 88.65 61)
-		(end 89.6 61.95)
+		(start 89.6 61.95)
+		(end 92.45 61.95)
 		(width 0.127)
 		(layer "B.Cu")
@@
 	)
 	(segment
-		(start 92.45 61.95)
-		(end 94.75 64.25)
+		(start 105.45 72.75)
+		(end 104.75 73.45)
 		(width 0.127)
 		(layer "B.Cu")
@@
 	)
 	(segment
-		(start 89.6 61.95)
-		(end 92.45 61.95)
+		(start 105.45 67.35)
+		(end 105.45 72.75)
 		(width 0.127)
 		(layer "B.Cu")
@@
 		(polygon
 			(pts
-				(xy 68.3 72.15) (xy 68.3 73.9) (xy 68.3 73.9) (xy 71.1 73.9) (xy 71.1 72.15) (xy 68.3 72.15)
+				(xy 68.3 72.15) (xy 68.3 73.9) (xy 71.1 73.9) (xy 71.1 72.15)
 			)
 		)

Commit message: PCB修改器件干涉问题，更换LED
Parts:
- removed D1: NCD0603G1, LED_SMD:LED_0603_1608Metric
- removed D2: NCD0603R1, LED_SMD:LED_0603_1608Metric
- removed D3: NCD0603B1, LED_SMD:LED_0603_1608Metric
- added D6: LED_RGBA, Library:LED_RGBA_1615, F.Cu at (65.8, 87.9)
- R36, R37, R38: moved to B.Cu
- moved R38 5.58 mm to (61.3, 86.2), turned to 90 degrees
- moved R37 3.93 mm to (62.3, 86.2), turned to 90 degrees
- moved R36 2.70 mm to (63.3, 86.2), turned to 90 degrees
- moved FB2 2.26 mm to (89.9, 64.2), turned to 0 degrees
Connections:
- net /GW5A_LV25MG121N/MCU_SWC renamed /GW5A_LV25MG121N/K9_MCU_SWC
- net /GW5A_LV25MG121N/MCU_SWD renamed /GW5A_LV25MG121N/L9_MCU_SWD
- R36 pad 1: +3V3 -> Net-(D6-RK)
- R36 pad 2: Net-(D1-A) -> /GW5A_LV25MG121N/L5_IOT63A
- R37 pad 1: +3V3 -> Net-(D6-GK)
- R37 pad 2: Net-(D2-A) -> /GW5A_LV25MG121N/J5_IOT61B
- R38 pad 1: +3V3 -> Net-(D6-BK)
- R38 pad 2: Net-(D3-A) -> /GW5A_LV25MG121N/H5_IOT61A
Routing:
- net Net-(D6-BK): track 0.00 -> 4.26 mm, vias 0 -> 1
- net /GW5A_LV25MG121N/H5_IOT61A: track 30.9 -> 26.8 mm, vias 2 -> 1
- net Net-(D6-RK): track 0.00 -> 3.92 mm, vias 0 -> 1
- net Net-(D6-GK): track 0.00 -> 3.47 mm, vias 0 -> 1
- net +3V3: track 135.3 -> 132.9 mm
- net /GW5A_LV25MG121N/J5_IOT61B: track 28.7 -> 26.7 mm, vias 2 -> 1
- net Net-(D3-A): track 1.49 -> 0.00 mm
- net Net-(D2-A): track 1.48 -> 0.00 mm
- net Net-(D1-A): track 1.47 -> 0.00 mm
- net /GW5A_LV25MG121N/L5_IOT63A: track 26.7 -> 26.6 mm, vias 2 -> 1

Commit message: 移植到新硬件
【PCB】输出端口串联33欧电阻，螺丝孔接地，串口RX上拉
【RTL】引脚适配，重构GPIO
【MCU】支持1115读取电压电流
Parts:
- added R39: 10K,1%, Resistor_SMD:R_0402_1005Metric, B.Cu at (93.0, 83.2)
- added R40: 33R,1%, Resistor_SMD:R_0402_1005Metric, B.Cu at (91.3, 71.3)
- added R41: 33R,1%, Resistor_SMD:R_0402_1005Metric, B.Cu at (91.3, 70.3)
- added R42: 33R,1%, Resistor_SMD:R_0402_1005Metric, B.Cu at (91.0, 62.5)
Connections:
- H1 pad 1: unconnected-(H1-Pad1) -> GND
- H2 pad 1: unconnected-(H2-Pad1) -> GND
- H3 pad 1: unconnected-(H3-Pad1) -> GND
- H4 pad 1: unconnected-(H4-Pad1) -> GND
- U13 pad 2: unconnected-(U13-A1-Pad2) -> GND
- U13 pad 6: /INTERFACE/UART_TX -> Net-(U13-B2)
- U5 pad 6: /INTERFACE/TDI -> Net-(U5-B2)
- U5 pad 7: /INTERFACE/TCK -> Net-(U5-B1)
Routing:
- net /INTERFACE/TDI: track 10.4 -> 4.76 mm
- net VTARG: track 108.0 -> 112.7 mm
- net /INTERFACE/UART_TX: track 29.0 -> 24.8 mm
- net /INTERFACE/TCK: track 8.51 -> 4.42 mm
- net Net-(U5-B2): track 0.00 -> 3.82 mm
- net Net-(U13-B2): track 0.00 -> 3.61 mm
- net Net-(U5-B1): track 0.00 -> 3.61 mm
- net /INTERFACE/UART_RX: track 22.8 -> 24.8 mm
- net GND: vias 52 -> 59
Other:
- board text removed: "JLCJLCJLCJLC"
