File: Hardware/plus/USB3320.kicad_sch (KiCad schematic)
At the start: 24 parts, among them J4 USB_C_Receptacle_USB2.0_16P, U1 ECMF02-2AMX6, U2 USB3320C-EZK

Commit message: 修改USB描述符驱动改为FPGA实现，解决部分电脑发送IN请求太快软核响应不及时导致的不识别USB的问题
Parts:
- R4, R5: 华秋编号 (none) -> G0064869; 立创编号 (none) -> C25905
Changed lines of the file:
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@@
+		(polyline
+			(pts
+				(xy 127 82.55) (xy 127 90.17) (xy 134.62 90.17) (xy 134.62 82.55) (xy 134.62 82.55)
+			)
+			(stroke
+				(width 0)
+				(type dash)
+			)
+			(fill
+				(type none)
+			)
+		)
+	)
+	(rule_area
 		(polyline
 			(pts
 				(xy 100.33 82.55) (xy 100.33 90.17) (xy 110.49 90.17) (xy 110.49 82.55) (xy 107.95 82.55)
-			)
-			(stroke
-				(width 0)
-				(type dash)
-			)
-			(fill
-				(type none)
-			)
-		)
-	)
-	(rule_area
-		(polyline
-			(pts
-				(xy 127 82.55) (xy 127 90.17) (xy 134.62 90.17) (xy 134.62 82.55) (xy 134.62 82.55)
 			)
 			(stroke
@@
 			)
 		)
+		(property "华秋编号" "G0064869"
+			(at 95.25 85.09 0)
+			(effects
+				(font
+					(size 1.27 1.27)
+				)
+				(hide yes)
+			)
+		)
+		(property "立创编号" "C25905"
+			(at 95.25 85.09 0)
+			(effects
+				(font
+					(size 1.27 1.27)
+				)
+				(hide yes)
+			)
+		)
 		(pin "2"
 		)
@@
 	)
 	(symbol
+		(lib_name "0402WGF5101TCE_1")
 		(lib_id "HPM6280Foc:0402WGF5101TCE")
 		(at 87.63 85.09 90)
@@
 			(at 87.63 85.09 0)
 			(effects
+				(font
+					(size 1.27 1.27)
+				)
+				(hide yes)
+			)
+		)
+		(property "华秋编号" "G0064869"
+			(at 87.63 85.09 0)
+			(effects
+				(font
+					(size 1.27 1.27)
+				)
+				(hide yes)
+			)
+		)
+		(property "立创编号" "C25905"
+			(at 87.63 85.09 0)
+			(effects
